File: CH32V003F4P6_BreakoutBoard.kicad_pcb (KiCad board)
At the start: 2 copper layers, 17.8 x 30.5 mm, 5 parts, among them J1 Conn_01x10_Pin, J2 Conn_01x10_Pin, J3 Conn_02x05_Odd_Even

Commit message: v2
Connections:
- J1 pad 2: Net-(J1-Pin_2) -> CH32V_TX_LinkE_RX
- J1 pad 3: Net-(J1-Pin_3) -> CH32V_RX_LinkE_TX
- J3 pad 7: unconnected-(J3-Pin_7-Pad7) -> CH32V_RX_LinkE_TX
- J3 pad 9: unconnected-(J3-Pin_9-Pad9) -> CH32V_TX_LinkE_RX
- U1 pad 2: Net-(J1-Pin_2) -> CH32V_TX_LinkE_RX
- U1 pad 3: Net-(J1-Pin_3) -> CH32V_RX_LinkE_TX
Routing:
- net CH32V_TX_LinkE_RX: track 0.00 -> 24.8 mm
- net CH32V_RX_LinkE_TX: track 0.00 -> 22.0 mm, vias 0 -> 1
- net Net-(J1-Pin_2): track 9.01 -> 0.00 mm
- net Net-(J1-Pin_3): track 7.19 -> 0.00 mm
Changed lines of the file:
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@@
   (net 2 "GND")
   (net 3 "Net-(J1-Pin_1)")
-  (net 4 "Net-(J1-Pin_2)")
-  (net 5 "Net-(J1-Pin_3)")
+  (net 4 "CH32V_TX_LinkE_RX")
+  (net 5 "CH32V_RX_LinkE_TX")
   (net 6 "Net-(J1-Pin_4)")
   (net 7 "Net-(J1-Pin_5)")
@@
   (net 21 "unconnected-(J3-Pin_3-Pad3)")
   (net 22 "unconnected-(J3-Pin_4-Pad4)")
-  (net 23 "unconnected-(J3-Pin_9-Pad9)")
-  (net 24 "unconnected-(J3-Pin_10-Pad10)")
-  (net 25 "unconnected-(J3-Pin_1-Pad1)")
-  (net 26 "unconnected-(J3-Pin_5-Pad5)")
-  (net 27 "unconnected-(J3-Pin_7-Pad7)")
+  (net 23 "unconnected-(J3-Pin_10-Pad10)")
+  (net 24 "unconnected-(J3-Pin_1-Pad1)")
+  (net 25 "unconnected-(J3-Pin_5-Pad5)")
   (footprint "Capacitor_SMD:C_0603_1608Metric" (layer "F.Cu")
     (at 129.54 91.44 -45)
@@
       (stroke (width 0.1) (type solid)) (layer "F.Fab"))
     (pad "1" thru_hole rect (at 0 0 90) (size 1.7 1.7) (drill 1) (layers "*.Cu" "*.Mask")
-      (net 25 "unconnected-(J3-Pin_1-Pad1)") (pinfunction "Pin_1") (pintype "passive+no_connect"))
+      (net 24 "unconnected-(J3-Pin_1-Pad1)") (pinfunction "Pin_1") (pintype "passive+no_connect"))
     (pad "2" thru_hole oval (at 2.54 0 90) (size 1.7 1.7) (drill 1) (layers "*.Cu" "*.Mask")
       (net 1 "5V") (pinfunction "Pin_2") (pintype "passive"))
@@
       (net 22 "unconnected-(J3-Pin_4-Pad4)") (pinfunction "Pin_4") (pintype "passive+no_connect"))
     (pad "5" thru_hole oval (at 0 5.08 90) (size 1.7 1.7) (drill 1) (layers "*.Cu" "*.Mask")
-      (net 26 "unconnected-(J3-Pin_5-Pad5)") (pinfunction "Pin_5") (pintype "passive+no_connect"))
+      (net 25 "unconnected-(J3-Pin_5-Pad5)") (pinfunction "Pin_5") (pintype "passive+no_connect"))
     (pad "6" thru_hole oval (at 2.54 5.08 90) (size 1.7 1.7) (drill 1) (layers "*.Cu" "*.Mask")
       (net 2 "GND") (pinfunction "Pin_6") (pintype "passive"))
     (pad "7" thru_hole oval (at 0 7.62 90) (size 1.7 1.7) (drill 1) (layers "*.Cu" "*.Mask")
-      (net 27 "unconnected-(J3-Pin_7-Pad7)") (pinfunction "Pin_7") (pintype "passive+no_connect"))
+      (net 5 "CH32V_RX_LinkE_TX") (pinfunction "Pin_7") (pintype "passive"))
     (pad "8" thru_hole oval (at 2.54 7.62 90) (size 1.7 1.7) (drill 1) (layers "*.Cu" "*.Mask")
       (net 13 "SWDIO") (pinfunction "Pin_8") (pintype "passive"))
     (pad "9" thru_hole oval (at 0 10.16 90) (size 1.7 1.7) (drill 1) (layers "*.Cu" "*.Mask")
-      (net 23 "unconnected-(J3-Pin_9-Pad9)") (pinfunction "Pin_9") (pintype "passive+no_connect"))
+      (net 4 "CH32V_TX_LinkE_RX") (pinfunction "Pin_9") (pintype "passive"))
     (pad "10" thru_hole oval (at 2.54 10.16 90) (size 1.7 1.7) (drill 1) (layers "*.Cu" "*.Mask")
-      (net 24 "unconnected-(J3-Pin_10-Pad10)") (pinfunction "Pin_10") (pintype "passive+no_connect"))
+      (net 23 "unconnected-(J3-Pin_10-Pad10)") (pinfunction "Pin_10") (pintype "passive+no_connect"))
     (model "${KICAD6_3DMODEL_DIR}/Connector_PinHeader_2.54mm.3dshapes/PinHeader_2x05_P2.54mm_Vertical.wrl"
       (offset (xyz 0 0 0))
@@
       (net 3 "Net-(J1-Pin_1)") (pinfunction "PD4/A7/UCK/T2CH1ETR/OPO/T1CH4ETR_") (pintype "bidirectional"))
     (pad "2" smd rect (at -2.9 -2.275) (size 1 0.4) (layers "F.Cu" "F.Paste" "F.Mask")
-      (net 4 "Net-(J1-Pin_2)") (pinfunction "PD5/A5/UTX/T2CH4_/URX_") (pintype "bidirectional"))
+      (net 4 "CH32V_TX_LinkE_RX") (pinfunction "PD5/A5/UTX/T2CH4_/URX_") (pintype "bidirectional"))
     (pad "3" smd rect (at -2.9 -1.625) (size 1 0.4) (layers "F.Cu" "F.Paste" "F.Mask")
-      (net 5 "Net-(J1-Pin_3)") (pinfunction "PD6/A6/URX/T2CH3_/UTX_") (pintype "bidirectional"))
+      (net 5 "CH32V_RX_LinkE_TX") (pinfunction "PD6/A6/URX/T2CH3_/UTX_") (pintype "bidirectional"))
     (pad "4" smd rect (at -2.9 -0.975) (size 1 0.4) (layers "F.Cu" "F.Paste" "F.Mask")
       (net 6 "Net-(J1-Pin_4)") (pinfunction "PD7/NRST/T2CH4/OPP1/UCK_") (pintype "bidirectional"))
@@
       (net 3 "Net-(J1-Pin_1)") (pinfunction "Pin_1") (pintype "passive"))
     (pad "2" thru_hole oval (at 0 -2.54 180) (size 1.7 1.7) (drill 1) (layers "*.Cu" "*.Mask")
-      (net 4 "Net-(J1-Pin_2)") (pinfunction "Pin_2") (pintype "passive"))
+      (net 4 "CH32V_TX_LinkE_RX") (pinfunction "Pin_2") (pintype "passive"))
     (pad "3" thru_hole oval (at 0 -5.08 180) (size 1.7 1.7) (drill 1) (layers "*.Cu" "*.Mask")
-      (net 5 "Net-(J1-Pin_3)") (pinfunction "Pin_3") (pintype "passive"))
+      (net 5 "CH32V_RX_LinkE_TX") (pinfunction "Pin_3") (pintype "passive"))
     (pad "4" thru_hole oval (at 0 -7.62 180) (size 1.7 1.7) (drill 1) (layers "*.Cu" "*.Mask")
       (net 6 "Net-(J1-Pin_4)") (pinfunction "Pin_4") (pintype "passive"))
@@
   (segment (start 130.81 82.55) (end 127 78.74) (width 0.25) (layer "F.Cu") (net 4))
   (segment (start 130.97 85.355) (end 130.81 85.195) (width 0.25) (layer "F.Cu") (net 4))
+  (segment (start 139.7 73.665) (end 134.62 78.745) (width 0.25) (layer "F.Cu") (net 4))
   (segment (start 130.81 85.195) (end 130.81 82.55) (width 0.25) (layer "F.Cu") (net 4))
+  (segment (start 134.62 83.82) (end 133.085 85.355) (width 0.25) (layer "F.Cu") (net 4))
   (segment (start 131.72 85.355) (end 130.97 85.355) (width 0.25) (layer "F.Cu") (net 4))
+  (segment (start 133.085 85.355) (end 131.72 85.355) (width 0.25) (layer "F.Cu") (net 4))
+  (segment (start 134.62 78.745) (end 134.62 83.82) (width 0.25) (layer "F.Cu") (net 4))
+  (segment (start 134.625 76.2) (end 129.54 76.2) (width 0.25) (layer "F.Cu") (net 5))
   (segment (start 130.846701 86.005) (end 130.36 85.518299) (width 0.25) (layer "F.Cu") (net 5))
   (segment (start 131.72 86.005) (end 130.846701 86.005) (width 0.25) (layer "F.Cu") (net 5))
   (segment (start 130.36 84.64) (end 127 81.28) (width 0.25) (layer "F.Cu") (net 5))
   (segment (start 130.36 85.518299) (end 130.36 84.64) (width 0.25) (layer "F.Cu") (net 5))
+  (segment (start 137.16 73.665) (end 134.625 76.2) (width 0.25) (layer "F.Cu") (net 5))
+  (via (at 129.54 76.2) (size 0.8) (drill 0.4) (layers "F.Cu" "B.Cu") (net 5))
+  (segment (start 129.54 76.2) (end 129.54 78.74) (width 0.25) (layer "B.Cu") (net 5))
+  (segment (start 129.54 78.74) (end 127 81.28) (width 0.25) (layer "B.Cu") (net 5))
   (segment (start 129.835 86.655) (end 127 83.82) (width 0.25) (layer "F.Cu") (net 6))
   (segment (start 131.72 86.655) (end 129.835 86.655) (width 0.25) (layer "F.Cu") (net 6))
