File: CH32V003F4P6_BreakoutBoard.kicad_sch (KiCad schematic)
At the start: 5 parts, among them J1 Conn_01x10_Pin, J2 Conn_01x10_Pin, J3 Conn_02x05_Odd_Even

Commit message: v2
Connections:
- net CH32V_TX_LinkE_RX: now reaches J1.2 (Pin_2), U1.2 (PD5/A5/UTX/T2CH4_/URX_)
- net CH32V_TX_LinkE_RX: now also J3.9 (Pin_9)
- net CH32V_RX_LinkE_TX: now reaches J1.3 (Pin_3), U1.3 (PD6/A6/URX/T2CH3_/UTX_)
- net CH32V_RX_LinkE_TX: now also J3.7 (Pin_7)
- no-connect marks 7 -> 5
Changed lines of the file:
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@@
   (junction (at 101.6 97.79) (diameter 0) (color 0 0 0 0)
+  )
+  (junction (at 101.6 82.55) (diameter 0) (color 0 0 0 0)
+  )
+  (junction (at 101.6 80.01) (diameter 0) (color 0 0 0 0)
   )
   (junction (at 101.6 92.71) (diameter 0) (color 0 0 0 0)
@@
   (no_connect (at 149.86 59.69))
   (no_connect (at 157.48 46.99))
-  (no_connect (at 154.94 59.69))
-  (no_connect (at 157.48 59.69))
   (no_connect (at 147.32 59.69))
   (wire (pts (xy 101.6 92.71) (xy 105.41 92.71))
@@
   )
   (wire (pts (xy 114.3 40.64) (xy 114.3 38.1))
+    (stroke (width 0) (type default))
+  )
+  (wire (pts (xy 154.94 59.69) (xy 154.94 63.5))
+    (stroke (width 0) (type default))
+  )
+  (wire (pts (xy 101.6 80.01) (xy 92.71 80.01))
     (stroke (width 0) (type default))
   )
@@
     (stroke (width 0) (type default))
   )
+  (wire (pts (xy 157.48 59.69) (xy 157.48 63.5))
+    (stroke (width 0) (type default))
+  )
   (wire (pts (xy 203.2 82.55) (xy 212.09 82.55))
     (stroke (width 0) (type default))
@@
   )
   (wire (pts (xy 199.39 85.09) (xy 203.2 85.09))
+    (stroke (width 0) (type default))
+  )
+  (wire (pts (xy 101.6 82.55) (xy 92.71 82.55))
     (stroke (width 0) (type default))
   )
@@
     )
   )
+  (global_label "CH32V_RX_LinkE_TX" (shape bidirectional) (at 154.94 63.5 180) (fields_autoplaced)
+    (effects (font (size 1.27 1.27)) (justify right))
+    (property "Intersheetrefs" "${INTERSHEET_REFS}" (at 132.2964 63.5 0)
+      (effects (font (size 1.27 1.27)) (justify right) hide)
+    )
+  )
+  (global_label "CH32V_TX_LinkE_RX" (shape bidirectional) (at 92.71 80.01 180) (fields_autoplaced)
+    (effects (font (size 1.27 1.27)) (justify right))
+    (property "Intersheetrefs" "${INTERSHEET_REFS}" (at 70.0664 80.01 0)
+      (effects (font (size 1.27 1.27)) (justify right) hide)
+    )
+  )
   (global_label "5V" (shape bidirectional) (at 147.32 44.45 90) (fields_autoplaced)
     (effects (font (size 1.27 1.27)) (justify left))
     (property "Intersheetrefs" "${INTERSHEET_REFS}" (at 147.32 38.1348 90)
       (effects (font (size 1.27 1.27)) (justify left) hide)
+    )
+  )
+  (global_label "CH32V_RX_LinkE_TX" (shape bidirectional) (at 92.71 82.55 180) (fields_autoplaced)
+    (effects (font (size 1.27 1.27)) (justify right))
+    (property "Intersheetrefs" "${INTERSHEET_REFS}" (at 70.0664 82.55 0)
+      (effects (font (size 1.27 1.27)) (justify right) hide)
     )
   )
@@
       (effects (font (size 1.27 1.27)) (justify left) hide)
     )
+  )
+  (global_label "CH32V_TX_LinkE_RX" (shape bidirectional) (at 157.48 63.5 0) (fields_autoplaced)
+    (effects (font (size 1.27 1.27)) (justify left))
+    (property "Intersheetrefs" "${INTERSHEET_REFS}" (at 180.1236 63.5 0)
+      (effects (font (size 1.27 1.27)) (justify left) hide)
+    )
